File: hardware/kicad/beta-main/sensors.kicad_sch (KiCad schematic)
At the start: 2 parts, among them U6 BNO086

Commit message: BNO086 tweaked
Parts:
- U6: symbol BNO086:BNO086 -> Beta:BNO086
Connections:
- now unconnected: U6.1 (RESV_NC), U6.12 (RESV_NC), U6.13 (RESV_NC), U6.21 (RESV_NC), U6.22 (RESV_NC), U6.23 (RESV_NC), U6.24 (RESV_NC), U6.7 (RESV_NC), U6.8 (RESV_NC)
Changed lines of the file:
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@@
 	)
 	(symbol
-		(lib_id "BNO086:BNO086")
+		(lib_id "Beta:BNO086")
 		(at 115.57 69.85 180)
 		(unit 1)
@@
 		(fields_autoplaced yes)
 		(property "Reference" "U6"
-			(at 115.57 95.25 0)
+			(at 115.57 41.91 0)
 			(effects
 				(font
@@
 		)
 		(property "Value" "BNO086"
-			(at 115.57 92.71 0)
+			(at 115.57 44.45 0)
 			(effects
 				(font
