File: hardware/kicad/beta-main/peripherals.kicad_sch (KiCad schematic)
At the start: 23 parts, among them J10 Servo Socket, J11 Servo Socket, J12 Servo Socket, J13 Servo Socket, J14 Conn_01x04_Pin, J15 Conn_01x04_Pin, J16 Conn_01x04_Pin, J17 Conn_01x04_Pin, J19 FAN0, J20 FAN1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

Commit message: add filled zones and layout 5V and 3V3
Parts:
- C1: footprint Capacitor_SMD:C_0603_1608Metric_Pad1.08x0.95mm_HandSolder -> Capacitor_SMD:C_0603_1608Metric
- R1, R2, R3, R4, R5: footprint Resistor_SMD:R_0402_1005Metric -> Resistor_SMD:R_0603_1608Metric

Commit message: sync
Parts:
- added R14: 10k, Resistor_SMD:R_0603_1608Metric, symbol Device:R
Connections:
- net +3V3: now also U3.10 (CLKSEL0), R14.1; no longer U3.18 (~{H_CS}), U3.4 (~{BOOT})
- net GND: now also U3.26 (XOUT32/CLKSEL1); no longer U3.10 (CLKSEL0)
- new net: R14.2, U3.4 (~{BOOT})
- no-connect marks 4 -> 3
Changed lines of the file:
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@@
 	)
 	(junction
-		(at 132.08 50.8)
-		(diameter 0)
-		(color 0 0 0 0)
-	)
-	(junction
 		(at 243.84 118.11)
 		(diameter 0)
@@
 	)
 	(no_connect
-		(at 69.85 66.04)
-	)
-	(no_connect
 		(at 69.85 68.58)
 	)
@@
 	(wire
 		(pts
-			(xy 130.81 50.8) (xy 132.08 50.8)
-		)
-		(stroke
-			(width 0)
-			(type default)
-		)
-	)
-	(wire
-		(pts
 			(xy 69.85 73.66) (xy 68.58 73.66)
 		)
@@
 	(wire
 		(pts
-			(xy 142.24 55.88) (xy 142.24 58.42)
-		)
-		(stroke
-			(width 0)
-			(type default)
-		)
-	)
-	(wire
-		(pts
 			(xy 33.02 114.3) (xy 50.8 114.3)
 		)
@@
 	(wire
 		(pts
-			(xy 132.08 50.8) (xy 132.08 53.34)
+			(xy 200.66 128.27) (xy 205.74 128.27)
 		)
 		(stroke
@@
 	(wire
 		(pts
-			(xy 200.66 128.27) (xy 205.74 128.27)
+			(xy 144.78 151.13) (xy 144.78 149.86)
 		)
 		(stroke
@@
 	(wire
 		(pts
-			(xy 144.78 151.13) (xy 144.78 149.86)
+			(xy 200.66 49.53) (xy 200.66 48.26)
 		)
 		(stroke
@@
 	(wire
 		(pts
-			(xy 200.66 49.53) (xy 200.66 48.26)
+			(xy 200.66 64.77) (xy 201.93 64.77)
 		)
 		(stroke
@@
 	(wire
 		(pts
-			(xy 200.66 64.77) (xy 201.93 64.77)
+			(xy 33.02 134.62) (xy 36.83 134.62)
 		)
 		(stroke
@@
 	(wire
 		(pts
-			(xy 33.02 134.62) (xy 36.83 134.62)
+			(xy 200.66 48.26) (xy 201.93 48.26)
 		)
 		(stroke
@@
 	(wire
 		(pts
-			(xy 200.66 48.26) (xy 201.93 48.26)
+			(xy 62.23 38.1) (xy 62.23 40.64)
 		)
 		(stroke
@@
 	(wire
 		(pts
-			(xy 62.23 38.1) (xy 62.23 40.64)
+			(xy 66.04 66.04) (xy 69.85 66.04)
 		)
 		(stroke
@@
 	(wire
 		(pts
-			(xy 133.35 46.99) (xy 133.35 48.26)
+			(xy 133.35 46.99) (xy 133.35 50.8)
 		)
 		(stroke
@@
 	(wire
 		(pts
-			(xy 142.24 58.42) (xy 130.81 58.42)
+			(xy 144.78 58.42) (xy 130.81 58.42)
 		)
 		(stroke
@@
 	(wire
 		(pts
+			(xy 133.35 50.8) (xy 130.81 50.8)
+		)
+		(stroke
+			(width 0)
+			(type default)
+		)
+	)
+	(wire
+		(pts
 			(xy 205.74 137.16) (xy 205.74 138.43)
 		)
@@
 	(wire
 		(pts
-			(xy 134.62 50.8) (xy 134.62 52.07)
+			(xy 134.62 53.34) (xy 134.62 54.61)
 		)
 		(stroke
@@
 	(wire
 		(pts
-			(xy 132.08 50.8) (xy 134.62 50.8)
+			(xy 132.08 53.34) (xy 134.62 53.34)
 		)
 		(stroke
@@
 	(wire
 		(pts
-			(xy 234.95 128.27) (xy 234.95 130.81)
+			(xy 144.78 57.15) (xy 144.78 58.42)
 		)
 		(stroke
@@
 	(wire
 		(pts
-			(xy 67.31 40.64) (xy 69.85 40.64)
+			(xy 234.95 128.27) (xy 234.95 130.81)
 		)
 		(stroke
@@
 	(wire
 		(pts
-			(xy 151.13 132.08) (xy 152.4 132.08)
+			(xy 67.31 40.64) (xy 69.85 40.64)
 		)
 		(stroke
@@
 	(wire
 		(pts
-			(xy 50.8 124.46) (xy 50.8 127)
+			(xy 151.13 132.08) (xy 152.4 132.08)
 		)
 		(stroke
@@
 	(wire
 		(pts
-			(xy 227.33 49.53) (xy 227.33 48.26)
+			(xy 50.8 124.46) (xy 50.8 127)
 		)
 		(stroke
@@
 	(wire
 		(pts
-			(xy 132.08 53.34) (xy 132.08 55.88)
+			(xy 227.33 49.53) (xy 227.33 48.26)
 		)
 		(stroke
@@
 	(wire
 		(pts
-			(xy 133.35 48.26) (xy 130.81 48.26)
+			(xy 132.08 53.34) (xy 132.08 55.88)
 		)
 		(stroke
@@
 	(wire
 		(pts
+			(xy 144.78 48.26) (xy 144.78 49.53)
+		)
+		(stroke
+			(width 0)
+			(type default)
+		)
+	)
+	(wire
+		(pts
 			(xy 144.78 149.86) (xy 152.4 149.86)
 		)
@@
 	(wire
 		(pts
+			(xy 66.04 67.31) (xy 66.04 66.04)
+		)
+		(stroke
+			(width 0)
+			(type default)
+		)
+	)
+	(wire
+		(pts
 			(xy 50.8 127) (xy 49.53 127)
 		)
@@
 	)
 	(symbol
+		(lib_id "Device:R")
+		(at 144.78 53.34 0)
+		(unit 1)
+		(exclude_from_sim no)
+		(in_bom yes)
+		(on_board yes)
+		(dnp no)
+		(property "Reference" "R14"
+			(at 147.32 52.0699 0)
+			(effects
+				(font
+					(size 1.27 1.27)
+				)
+				(justify left)
+			)
+		)
+		(property "Value" "10k"
+			(at 147.32 54.6099 0)
+			(effects
+				(font
+					(size 1.27 1.27)
+				)
+				(justify left)
+			)
+		)
+		(property "Footprint" "Resistor_SMD:R_0603_1608Metric"
+			(at 143.002 53.34 90)
+			(effects
+				(font
+					(size 1.27 1.27)
+				)
+				(hide yes)
+			)
+		)
+		(property "Datasheet" "~"
+			(at 144.78 53.34 0)
+			(effects
+				(font
+					(size 1.27 1.27)
+				)
+				(hide yes)
+			)
+		)
+		(property "Description" "Resistor"
+			(at 144.78 53.34 0)
+			(effects
+				(font
+					(size 1.27 1.27)
+				)
+				(hide yes)
+			)
+		)
+		(property "Sim.Device" ""
+			(at 144.78 53.34 0)
+			(effects
+				(font
+					(size 1.27 1.27)
+				)
+				(hide yes)
+			)
+		)
+		(property "Sim.Pins" ""
+			(at 144.78 53.34 0)
+			(effects
+				(font
+					(size 1.27 1.27)
+				)
+				(hide yes)
+			)
+		)
+		(property "Sim.Type" ""
+			(at 144.78 53.34 0)
+			(effects
+				(font
+					(size 1.27 1.27)
+				)
+				(hide yes)
+			)
+		)
+		(pin "2"
+		)
+		(pin "1"
+		)
+		(instances
+			(project "beta-main"
+				(path "/6834c9e9-3e61-4f01-9d2c-ccd95d8f63cf/eb97c806-c815-45d1-bff9-8ccc678dc3c5"
+					(reference "R14")
+					(unit 1)
+				)
+			)
+		)
+	)
+	(symbol
 		(lib_id "power:+3V3")
 		(at 123.19 114.3 0)
@@
 	(symbol
 		(lib_id "power:GND")
-		(at 134.62 52.07 0)
+		(at 134.62 54.61 0)
 		(unit 1)
 		(exclude_from_sim no)
@@
 		(on_board yes)
 		(dnp no)
-		(fields_autoplaced yes)
 		(property "Reference" "#PWR078"
-			(at 134.62 58.42 0)
+			(at 134.62 60.96 0)
 			(effects
 				(font
@@
 		)
 		(property "Value" "GND"
-			(at 137.16 53.3399 0)
+			(at 137.16 55.8799 0)
 			(effects
 				(font
@@
 		)
 		(property "Footprint" ""
-			(at 134.62 52.07 0)
+			(at 134.62 54.61 0)
 			(effects
 				(font
@@
 		)
 		(property "Datasheet" ""
-			(at 134.62 52.07 0)
+			(at 134.62 54.61 0)
 			(effects
 				(font
@@
 		)
 		(property "Description" "Power symbol creates a global label with name \"GND\" , ground"
-			(at 134.62 52.07 0)
+			(at 134.62 54.61 0)
 			(effects
 				(font
@@
 	(symbol
 		(lib_id "power:+3V3")
-		(at 142.24 55.88 0)
+		(at 144.78 48.26 0)
 		(unit 1)
 		(exclude_from_sim no)
@@
 		(fields_autoplaced yes)
 		(property "Reference" "#PWR079"
-			(at 142.24 59.69 0)
+			(at 144.78 52.07 0)
 			(effects
 				(font
@@
 		)
 		(property "Value" "+3V3"
-			(at 144.78 54.6099 0)
+			(at 147.32 46.9899 0)
 			(effects
 				(font
@@
 		)
 		(property "Footprint" ""
-			(at 142.24 55.88 0)
+			(at 144.78 48.26 0)
 			(effects
 				(font
@@
 		)
 		(property "Datasheet" ""
-			(at 142.24 55.88 0)
+			(at 144.78 48.26 0)
 			(effects
 				(font
@@
 		)
 		(property "Description" "Power symbol creates a global label with name \"+3V3\""
-			(at 142.24 55.88 0)
+			(at 144.78 48.26 0)
 			(effects
 				(font
@@
 					(unit 1)
 				)
+			)
+		)
+	)
+	(symbol
+		(lib_id "power:GND")
+		(at 66.04 67.31 0)
+		(mirror y)
+		(unit 1)
+		(exclude_from_sim no)
+		(in_bom yes)
+		(on_board yes)
+		(dnp no)
+		(property "Reference" "#PWR0140"
+			(at 66.04 73.66 0)
+			(effects
+				(font
+					(size 1.27 1.27)
+				)
+				(hide yes)
+			)
+		)
+		(property "Value" "GND"
+			(at 63.5 68.5799 0)
+			(effects
+				(font
+					(size 1.27 1.27)
+				)
+				(justify left)
+			)
+		)
+		(property "Footprint" ""
+			(at 66.04 67.31 0)
+			(effects
+				(font
+					(size 1.27 1.27)
+				)
+				(hide yes)
+			)
+		)
+		(property "Datasheet" ""
+			(at 66.04 67.31 0)
+			(effects
+				(font
+					(size 1.27 1.27)
+				)
+				(hide yes)
+			)
+		)
+		(property "Description" "Power symbol creates a global label with name \"GND\" , ground"
+			(at 66.04 67.31 0)
+			(effects
+				(font
+					(size 1.27 1.27)
+				)
+				(hide yes)
+			)
+		)
+		(pin "1"
+		)
+		(instances
+			(project "beta-main"
+				(path "/6834c9e9-3e61-4f01-9d2c-ccd95d8f63cf/eb97c806-c815-45d1-bff9-8ccc678dc3c5"
+					(reference "#PWR0140")
+					(unit 1)
+				)
