File: hardware/kicad/beta-main/peripherals.kicad_sch (KiCad schematic)
At the start: 24 parts, among them J10 Servo Socket, J11 Servo Socket, J12 Servo Socket, J13 Servo Socket, J14 Conn_01x04_Pin, J15 Conn_01x04_Pin, J16 Conn_01x04_Pin, J17 Conn_01x04_Pin, J19 FAN0, J20 FAN1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

Commit message: resolve DRC issues and generate fab files
Parts:
- added C22, C23: 0.1u, Capacitor_SMD:C_0603_1608Metric, symbol Device:C
- added J24, J25: FAN1, Connector_JST:JST_PH_B2B-PH-K_1x02_P2.00mm_Vertical, symbol Connector:Conn_01x02_Pin
- added JP1: SolderJumper_2_Open, BETA:SolderJumper-2, symbol Jumper:SolderJumper_2_Open
- added R15: 2.2k, Resistor_SMD:R_0603_1608Metric, symbol Device:R
- added R16: 10k, Resistor_SMD:R_0603_1608Metric, symbol Device:R
Connections:
- net BNO_RST is gone; now on net +3V3: U3.11 (~{RST})
- net +3V3: now also C22.1, C23.1, R15.1, R16.1
- net +BATT: now also J24.1 (Pin_1), J25.1 (Pin_1)
- net BNO_SCL: now also R15.2
- net BNO_SDA: now also R16.2
- net GND: now also C22.2, C23.2, JP1.2 (B)
- net at D2.1 (K), J19.2 (Pin_2), J20.2 (Pin_2)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: now also J24.2 (Pin_2), J25.2 (Pin_2)
- net at R14.2, U3.4 (~{BOOT}): now also JP1.1 (A)
- no-connect marks 3 -> 4
Other:
- moved on the sheet: D2, R13, R14

Commit message: sync changes
Other:
- moved on the sheet: D2, J19, J20, J24, J25, Q2, R13

Commit message: sync
Parts:
- J14, J15, J16, J17: MP (none) -> S4B-PH-K
Changed lines of the file:
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@@
 			)
 		)
+		(property "MP" "S4B-PH-K"
+			(at 233.68 64.77 0)
+			(effects
+				(font
+					(size 1.27 1.27)
+				)
+				(hide yes)
+			)
+		)
 		(pin "4"
 		)
@@
 			)
 		)
+		(property "MP" "S4B-PH-K"
+			(at 207.01 64.77 0)
+			(effects
+				(font
+					(size 1.27 1.27)
+				)
+				(hide yes)
+			)
+		)
 		(pin "4"
 		)
@@
 			)
 		)
+		(property "MP" "S4B-PH-K"
+			(at 233.68 43.18 0)
+			(effects
+				(font
+					(size 1.27 1.27)
+				)
+				(hide yes)
+			)
+		)
 		(pin "4"
 		)
@@
 			(at 207.01 43.18 0)
 			(effects
+				(font
+					(size 1.27 1.27)
+				)
+				(hide yes)
+			)
+		)
+		(property "MP" "S4B-PH-K"
+			(at 207.01 43.18 0)
+			(effects

Commit message: add final touches, generate rev A fab and step files
Parts:
- added C2, C24: 100u, Capacitor_SMD:CP_Elec_6.3x5.7, symbol Device:C_Polarized
- J10, J11, J12, J13: value Servo Socket -> Conn_01x03_Pin; footprint Connector_JST:JST_XH_S3B-XH-A_1x03_P2.50mm_Horizontal -> Connector_JST:JST_XH_B3B-XH-A_1x03_P2.50mm_Vertical
- J14, J15, J16, J17: footprint Connector_JST:JST_PH_S4B-PH-K_1x04_P2.00mm_Horizontal -> Connector_JST:JST_PH_B4B-PH-K_1x04_P2.00mm_Vertical
- J19: value FAN0 -> Conn_01x02_Pin
- J20, J24, J25: value FAN1 -> Conn_01x02_Pin
- R15: value 2.2k -> 10k
Connections:
- net +BATT: now also C2.1, C24.1
- net GND: now also C2.2, C24.2
Other:
- moved on the sheet: D2, J19, J20, J24, J25, Q2, R13
